Commit message: trying using already available rovers

File: urdf/rover.urdf.xacro (robot description, xacro)
@@ -1,106 +1,180 @@
-<?xml version="1.0" ?>
-<robot name="rover">
+<?xml version="1.0"?>
+<robot xmlns:xacro="http://www.ros.org/wiki/xacro" name="rover">
+  <xacro:property name="base_width" value="0.16"/>
+  <xacro:property name="base_len" value="0.16"/>
+  <xacro:property name="wheel_radius" value="0.035"/>
+  <xacro:property name="base_wheel_gap" value="0.007"/>
+  <xacro:property name="wheel_separation" value="0.15"/>
+  <xacro:property name="wheel_joint_offset" value="0.02"/>
+  <xacro:property name="caster_wheel_radius" value="${wheel_radius/2}"/>
+  <xacro:property name="caster_wheel_mass" value="0.001"/>
+  <xacro:property name="caster_wheel_joint_offset" value="-0.052"/>
+  <!--Color Properties-->
+  <material name="blue">
+    <color rgba="0 0 0.8 1"/>
+  </material>
+  <material name="black">
+    <color rgba="0 0 0 1"/>
+  </material>
+  <material name="white">
+    <color rgba="1 1 1 1"/>
+  </material>
+  <material name="red">
+    <color rgba="0.8 0.0 0.0 1.0"/>
+  </material>
+  <!--Interial macros-->
+  <xacro:macro name="cylinder_inertia" params="m r h">
+    <inertial>
+      <mass value="${m}"/>
+      <inertia ixx="${m*(3*r*r+h*h)/12}" ixy = "0" ixz = "0" iyy="${m*(3*r*r+h*h)/12}" iyz = "0" izz="${m*r*r/2}"/>
+    </inertial>
+  </xacro:macro>
+  <xacro:macro name="box_inertia" params="m w h d">
+    <inertial>
+      <mass value="${m}"/>
+      <inertia ixx="${m / 12.0 * (d*d + h*h)}" ixy="0.0" ixz="0.0" iyy="${m / 12.0 * (w*w + h*h)}" iyz="0.0" izz="${m / 12.0 * (w*w + d*d)}"/>
+    </inertial>
+  </xacro:macro>
+  <xacro:macro name="sphere_inertia" params="m r">
+    <inertial>
+      <mass value="${m}"/>
+      <inertia ixx="${2.0*m*(r*r)/5.0}" ixy="0.0" ixz="0.0" iyy="${2.0*m*(r*r)/5.0}" iyz="0.0" izz="${2.0*m*(r*r)/5.0}"/>
+    </inertial>
+  </xacro:macro>
+  <!--Base Footprint-->
+  <link name="base_footprint">
+    <xacro:box_inertia m="10" w="0.001" h="0.001" d="0.001"/>
+    <visual>
+        <origin xyz="0 0 0" rpy="0 0 0" />
+        <geometry>
+            <box size="0.001 0.001 0.001" />
+        </geometry>
+    </visual>
+  </link>
+  <!--Base link-->
   <link name="base_link">
+    <xacro:box_inertia m="10" w="${base_len}" h="${base_width}" d="0.01"/>
     <visual>
       <geometry>
-        <box size="0.5 0.3 0.2"/>
+        <box size="${base_len} ${base_width} 0.01"/>
       </geometry>
-      <material>
-        <color rgba="1 0 0 1"/> <!-- Changed to red for better visibility -->
-      </material>
+      <material name="black"/>
     </visual>
     <collision>
       <geometry>
-        <box size="0.5 0.3 0.2"/>
+        <box size="${base_len} ${base_width} 0.01"/>
       </geometry>
     </collision>
   </link>
-  <!-- Front Left Wheel -->
-  <joint name="base_to_front_left_wheel" type="continuous">
-    <parent link="base_link"/>
-    <child link="front_left_wheel"/>
-    <origin xyz="0.2 0.15 -0.1" rpy="0 0 0"/>
-    <axis xyz="0 1 0"/>
+  <!--base_link to base_footprint Joint-->
+  <joint name="base_link_joint" type="fixed">
+    <origin xyz="0 0 ${wheel_radius + 0.005}" rpy="0 0 0" />
+    <parent link="base_footprint"/>
+    <child link="base_link" />
   </joint>
-  <link name="front_left_wheel">
+  <!--Wheel link & joint macro-->
+  <xacro:macro name="wheel" params="prefix reflect">
+    <link name="${prefix}_wheel">
+      <visual>
+        <origin xyz="0 0 0" rpy="${pi/2} 0 0"/>
+        <geometry>
+          <cylinder radius="${wheel_radius}" length="0.005"/>
+        </geometry>
+        <material name="red"/>
+      </visual>
+      <collision>
+        <origin xyz="0 0 0" rpy="${pi/2} 0 0"/>
+        <geometry>
+          <cylinder radius="${wheel_radius}" length="0.005"/>
+        </geometry>
+      </collision>
+      <xacro:cylinder_inertia m="10" r="${wheel_radius}" h="0.005"/>
+    </link>
+    <joint name="${prefix}_wheel_joint" type="continuous">
+      <axis xyz="0 1 0" rpy="0 0 0" />
+      <parent link="base_link"/>
+      <child link="${prefix}_wheel"/>
+      <origin xyz="${wheel_joint_offset} ${((base_width/2)+base_wheel_gap)*reflect} -0.005" rpy="0 0 0"/>
+    </joint>
+  </xacro:macro>
+  <!--Create Left & Right Wheel links/joints-->
+  <xacro:wheel prefix="left" reflect="1"/>
+  <xacro:wheel prefix="right" reflect="-1"/>
+  <!--Caster Wheel Link-->
+  <link name="caster_wheel">
     <visual>
+      <origin xyz="0 0 0" rpy="0 0 0"/>
       <geometry>
-        <cylinder radius="0.05" length="0.02"/>
+        <sphere radius="${caster_wheel_radius}"/>
       </geometry>
-      <material>
-        <color rgba="0 0 0 1"/>
-      </material>
+      <material name="blue"/>
     </visual>
     <collision>
+      <origin xyz="0 0 0" rpy="0 0 0"/>
       <geometry>
-        <cylinder radius="0.05" length="0.02"/>
+        <sphere radius="${caster_wheel_radius}"/>
       </geometry>
     </collision>
+    <xacro:sphere_inertia m="10" r="${caster_wheel_radius}"/>
   </link>
-  <!-- Front Right Wheel -->
-  <joint name="base_to_front_right_wheel" type="continuous">
+  <!--Caster Wheel Joint-->
+  <joint name="caster_wheel_joint" type="continuous">
+    <axis xyz="0 1 0" rpy="0 0 0" />
     <parent link="base_link"/>
-    <child link="front_right_wheel"/>
-    <origin xyz="0.2 -0.15 -0.1" rpy="0 0 0"/>
-    <axis xyz="0 1 0"/>
+    <child link="caster_wheel"/>
+    <origin xyz="${caster_wheel_joint_offset} 0 -${caster_wheel_radius+0.005}" rpy="0 0 0"/>
   </joint>
-  <link name="front_right_wheel">
-    <visual>
-      <geometry>
-        <cylinder radius="0.05" length="0.02"/>
-      </geometry>
-      <material>
-        <color rgba="0 0 0 1"/>
-      </material>
-    </visual>
-    <collision>
-      <geometry>
-        <cylinder radius="0.05" length="0.02"/>
-      </geometry>
-    </collision>
-  </link>
-  <!-- Rear Left Wheel -->
-  <joint name="base_to_rear_left_wheel" type="continuous">
-    <parent link="base_link"/>
-    <child link="rear_left_wheel"/>
-    <origin xyz="-0.2 0.15 -0.1" rpy="0 0 0"/>
-    <axis xyz="0 1 0"/>
-  </joint>
-  <link name="rear_left_wheel">
-    <visual>
-      <geometry>
-        <cylinder radius="0.05" length="0.02"/>
-      </geometry>
-      <material>
-        <color rgba="0 0 0 1"/>
-      </material>
-    </visual>
-    <collision>
-      <geometry>
-        <cylinder radius="0.05" length="0.02"/>
-      </geometry>
-    </collision>
-  </link>
-  <!-- Rear Right Wheel -->
-  <joint name="base_to_rear_right_wheel" type="continuous">
-    <parent link="base_link"/>
-    <child link="rear_right_wheel"/>
-    <origin xyz="-0.2 -0.15 -0.1" rpy="0 0 0"/>
-    <axis xyz="0 1 0"/>
-  </joint>
-  <link name="rear_right_wheel">
-    <visual>
-      <geometry>
-        <cylinder radius="0.05" length="0.02"/>
-      </geometry>
-      <material>
-        <color rgba="0 0 0 1"/>
-      </material>
-    </visual>
-    <collision>
-      <geometry>
-        <cylinder radius="0.05" length="0.02"/>
-      </geometry>
-    </collision>
-  </link>
+<!-- laser -->
+<link name="laser">
+  <xacro:cylinder_inertia m="5" r="0.025" h="0.025"/>
+  <visual>
+    <geometry>
+      <cylinder radius="0.025" length="0.025"/>
+     </geometry>
+  </visual>
+  <collision>
+    <origin/>
+    <geometry>
+      <cylinder radius="0.025" length="0.025"/>
+    </geometry>
+  </collision>
+</link>
+<joint name="laser_joint" type="fixed">
+  <origin xyz="0 0.0 0.015" rpy="0.0 0.0 3.14"/>
+  <axis xyz="0 0 1" />
+  <parent link="base_link"/>
+  <child link="laser"/>
+</joint>
+<gazebo reference="laser">
+  <sensor type="ray" name="laser">
+      <pose>0 0 0 0 0 0</pose>
+      <visualize>false</visualize>
+      <update_rate>40</update_rate>
+      <ray>
+          <scan>
+              <horizontal>
+                  <samples>1440</samples>
+                  <resolution>0.5</resolution>
+                  <min_angle>-1.578</min_angle>
+                  <max_angle>1.578</max_angle>
+              </horizontal>
+          </scan>
+          <range>
+            <min>0.10</min>
+            <max>3.0</max>
+            <resolution>0.01</resolution>
+          </range>
+          <noise>
+            <type>gaussian</type>
+            <mean>0.0</mean>
+            <stddev>0.01</stddev>
+          </noise>
+      </ray>
+      <plugin name="laser_controller" filename="libgazebo_ros_laser.so">
+          <topicName>/scan</topicName>
+          <frameName>laser</frameName>
+      </plugin>
+  </sensor>
+</gazebo>
+  <xacro:include filename="$(find pde4430_ex2)/urdf/rover_gazebo_plugins.xacro"/>
 </robot>
